Commit message: adjust urdf for kinematics calculation and add gitignore

File: tinyquad_urdf/urdf/tiny_quad.urdf (robot description, URDF)
Before this commit: robot tiny_quad, 17 links, 16 joints
Links:
- added link base_footprint
- link LBL_L: geometry 
- link LFL_L: geometry 
- link RBL_L: geometry 
- link RBS_L: mass 0 -> 0.0576835055796688
- link RFL_L: geometry 
Joints:
- added joint base_joint: type fixed, parent base_footprint, child base_link, origin xyz=0 0 0 rpy=0 0 0
- joint LBC_J: origin xyz=2.0629E-05 0.012 -0.085 rpy=0 0 0 -> xyz=2.0629E-05 0 -0.085 rpy=0 0 0
- joint LBL_J: limit lower=0 upper=0 effort=0 velocity=0 -> lower=-1.5708 upper=1.1 effort=1.0787315 velocity=7.48; mimic joint=LFS_J multiplier=1 offset=0 -> (none); origin xyz=0 0.01675 -0.078388 rpy=0 0 0 -> xyz=0 0 -0.078388 rpy=0 0 0
- joint LBS_J: limit lower=0 upper=0 effort=0 velocity=0 -> lower=0 upper=1.5708 effort=1.0787315 velocity=7.48; mimic joint=LFS_J multiplier=1 offset=0 -> (none)
- joint LBU_J: limit lower=0 upper=0 effort=0 velocity=0 -> lower=0 upper=1 effort=1.0787315 velocity=7.48; mimic joint=LFS_J multiplier=1 offset=0 -> (none); origin xyz=-0.037107 0.01375 0 rpy=0 0 0 -> xyz=-0.037107 0 0 rpy=0 0 0
- joint LFC_J: origin xyz=2.0629E-05 0.012 -0.085 rpy=0 0 0 -> xyz=2.0629E-05 0 -0.085 rpy=0 0 0
- joint LFL_J: limit lower=0 upper=0 effort=0 velocity=0 -> lower=-1.1 upper=1.5708 effort=1.0787315 velocity=7.48; mimic joint=LFS_J multiplier=1 offset=0 -> (none); origin xyz=0 0.01675 -0.078388 rpy=0 0 0 -> xyz=0 0 -0.078388 rpy=0 0 0
- joint LFS_J: limit lower=-1.5708 upper=1.5708 effort=1.0787315 velocity=7.48 -> lower=0 upper=1.5708 effort=1.0787315 velocity=7.48
- joint LFU_J: limit lower=0 upper=0 effort=0 velocity=0 -> lower=-1 upper=0 effort=1.0787315 velocity=7.48; mimic joint=LFS_J multiplier=1 offset=0 -> (none); origin xyz=-0.037107 0.01375 0 rpy=0 0 0 -> xyz=-0.037107 0 0 rpy=0 0 0
- joint RBC_J: origin xyz=1.9364E-05 -0.012 -0.085 rpy=0 0 0 -> xyz=1.9364E-05 0 -0.085 rpy=0 0 0
- joint RBL_J: limit lower=0 upper=0 effort=0 velocity=0 -> lower=-1.1 upper=1.5708 effort=1.0787315 velocity=7.48; mimic joint=LFS_J multiplier=1 offset=0 -> (none); origin xyz=0 -0.01675 -0.078391 rpy=0 0 0 -> xyz=0 0 -0.078391 rpy=0 0 0
- joint RBS_J: limit lower=0 upper=0 effort=0 velocity=0 -> lower=0 upper=1.5708 effort=1.0787315 velocity=7.48; mimic joint=LFS_J multiplier=1 offset=0 -> (none)
- joint RBU_J: limit lower=0 upper=0 effort=0 velocity=0 -> lower=-1.1 upper=0 effort=1.0787315 velocity=7.48; mimic joint=LFS_J multiplier=1 offset=0 -> (none); origin xyz=-0.037107 -0.01375 0 rpy=0 0 0 -> xyz=-0.037107 0 0 rpy=0 0 0
- joint RFC_J: origin xyz=1.9364E-05 -0.012 -0.085 rpy=0 0 0 -> xyz=1.9364E-05 0 -0.085 rpy=0 0 0
- joint RFL_J: limit lower=0 upper=0 effort=0 velocity=0 -> lower=-1.1 upper=1.5708 effort=1.0787315 velocity=7.48; mimic joint=LFS_J multiplier=1 offset=0 -> (none); origin xyz=0 -0.01675 -0.078391 rpy=0 0 0 -> xyz=0 0 -0.078391 rpy=0 0 0
- joint RFS_J: limit lower=0 upper=0 effort=0 velocity=0 -> lower=-1.5708 upper=0 effort=1.0787315 velocity=7.48; mimic joint=LFS_J multiplier=1 offset=0 -> (none)
- joint RFU_J: limit lower=0 upper=0 effort=0 velocity=0 -> lower=0 upper=1.1 effort=1.0787315 velocity=7.48; mimic joint=LFS_J multiplier=1 offset=0 -> (none); origin xyz=-0.037107 -0.01375 0 rpy=0 0 0 -> xyz=-0.037107 0 0 rpy=0 0 0
