Commit message: add wheels and diff drive

File: tinyquad_description/urdf/tinyquad.urdf.xacro (robot description, xacro)
@@ -4,4 +4,5 @@
   <xacro:include filename="$(find tinyquad_description)/urdf/tinyquad_transmission.xacro" />
   <xacro:include filename="$(find tinyquad_description)/urdf/tinyquad_sensors.urdf.xacro" />
+  <xacro:include filename="$(find tinyquad_description)/urdf/tinyquad_wheel.xacro" />
   <xacro:tinyquad />
   <xacro:tinyquad_transmission name="LFS"/>
@@ -17,4 +18,10 @@
   <xacro:tinyquad_transmission name="RBU"/>
   <xacro:tinyquad_transmission name="RBL"/>
+  <xacro:tinyquad_wheel pose_prefix="LB" y_mirror="1"/>
+  <xacro:tinyquad_wheel pose_prefix="RB" y_mirror="-1"/>
+  <!-- <xacro:tinyquad_wheel pose_prefix="LB" y_mirror="1"/>
+  <xacro:tinyquad_wheel pose_prefix="RB" y_mirror="-1"/> -->
+  <xacro:tinyquad_wheel_transmission name="LB"/>
+  <xacro:tinyquad_wheel_transmission name="RB"/>
   <gazebo>
       <plugin name="gazebo_ros_control" filename="libgazebo_ros_control.so">

File: tinyquad_description/urdf/tinyquad_transmission.xacro (robot description, xacro)
@@ -12,3 +12,15 @@
     </transmission>
   </xacro:macro>
+  <xacro:macro name="tinyquad_wheel_transmission" params="name">
+    <transmission name="${name}_wheel_control">
+      <type>transmission_interface/SimpleTransmission</type>
+      <joint name="${name}_wheel_joint">
+        <hardwareInterface>hardware_interface/VelocityJointInterface</hardwareInterface>
+      </joint>
+      <actuator name="${name}_wheel_motor">
+        <hardwareInterface>hardware_interface/VelocityJointInterface</hardwareInterface>
+        <mechanicalReduction>1</mechanicalReduction>
+      </actuator>
+    </transmission>
+  </xacro:macro>
 </robot>
