Commit message: fix urdf bug and tune position pid control

File: tinyquad_description/urdf/tinyquad_frame.urdf.xacro (robot description, xacro)
@@ -159,8 +159,8 @@
         link="LFU_L" />
       <axis
-        xyz="0 -1 0" />
-      <limit
-        lower="-1"
-        upper="0"
+        xyz="0 1 0" />
+      <limit
+        lower="0"
+        upper="1.1"
         effort="1.0787315"
         velocity="7.48" />
@@ -221,8 +221,8 @@
         link="LFL_L" />
       <axis
-        xyz="0 -1 0" />
-      <limit
-        lower="-1.1"
-        upper="1.5708"
+        xyz="0 1 0" />
+      <limit
+        lower="-1.5708"
+        upper="1.1"
         effort="1.0787315"
         velocity="7.48" />
@@ -336,8 +336,8 @@
         link="RFS_L" />
       <axis
-        xyz="1 0 0" />
-      <limit
-        lower="-1.5708"
-        upper="0"
+        xyz="-1 0 0" />
+      <limit
+        lower="0"
+        upper="1.5708"
         effort="1.0787315"
         velocity="7.48" />
@@ -460,8 +460,8 @@
         link="RFL_L" />
       <axis
-        xyz="0 -1 0" />
-      <limit
-        lower="-1.1"
-        upper="1.5708"
+        xyz="0 1 0" />
+      <limit
+        lower="-1.5708"
+        upper="1.1"
         effort="1.0787315"
         velocity="7.48" />
@@ -640,5 +640,5 @@
       <limit
         lower="0"
-        upper="1"
+        upper="1.1"
         effort="1.0787315"
         velocity="7.48" />
@@ -876,8 +876,8 @@
         link="RBU_L" />
       <axis
-        xyz="0 -1 0" />
-      <limit
-        lower="-1.1"
-        upper="0"
+        xyz="0 1 0" />
+      <limit
+        lower="0"
+        upper="1.1"
         effort="1.0787315"
         velocity="7.48" />
@@ -938,8 +938,8 @@
         link="RBL_L" />
       <axis
-        xyz="0 -1 0" />
-      <limit
-        lower="-1.1"
-        upper="1.5708"
+        xyz="0 1 0" />
+      <limit
+        lower="-1.5708"
+        upper="1.1"
         effort="1.0787315"
         velocity="7.48" />

Commit message: complete single leg joint mode and add flexible contact joint

File: tinyquad_description/urdf/tinyquad_frame.urdf.xacro (robot description, xacro)
@@ -165,8 +165,4 @@
         effort="1.0787315"
         velocity="7.48" />
-      <!--mimic
-        joint="LFS_J"
-        multiplier="1"
-        offset="0" /-->
     </joint>
     <link
@@ -186,5 +182,5 @@
           izz="2.20436639521685E-05" />
       </inertial>
-      <!-- <visual>
+      <visual>
         <origin
           xyz="0 0.0305 0"
@@ -208,5 +204,5 @@
             filename="package://tinyquad_description/meshes/LFL_L.STL" />
         </geometry>
-      </collision> -->
+      </collision>
     </link>
     <joint
@@ -227,8 +223,4 @@
         effort="1.0787315"
         velocity="7.48" />
-      <!--mimic
-        joint="LFS_J"
-        multiplier="1"
-        offset="0" /-->
     </joint>
     <link
@@ -251,8 +243,7 @@
         <origin
           xyz="0 0.0425 0"
-          rpy="0 0 0" />
-        <geometry>
-          <mesh
-            filename="package://tinyquad_description/meshes/LFC_L.STL" />
+          rpy="1.5708 0 0" />
+        <geometry>
+          <cylinder radius="0.001" length="0.01"/>
         </geometry>
         <material
@@ -265,23 +256,16 @@
         <origin
           xyz="0 0.0425 0"
-          rpy="0 0 0" />
-        <geometry>
-          <mesh
-            filename="package://tinyquad_description/meshes/LFC_L.STL" />
-        </geometry>
-      </collision>
-    </link>
-    <joint
-      name="LFC_J"
-      type="fixed">
-      <origin
-        xyz="2.0629E-05 0 -0.085"
-        rpy="0 0 0" />
-      <parent
-        link="LFL_L" />
-      <child
-        link="LFC_L" />
-      <axis
-        xyz="0 0 0" />
+          rpy="1.5708 0 0" />
+        <geometry>
+            <cylinder radius="0.001" length="0.1"/>
+        </geometry>
+      </collision>
+    </link>
+    <joint name="LFC_J" type="revolute">
+      <origin xyz="2.0629E-05 0 -0.085" rpy="0 0 0" />
+      <limit lower="-3.141592" upper="3.141592" effort="1.0787315" velocity="7.48" />
+      <parent link="LFL_L" />
+      <child link="LFC_L" />
+      <axis xyz="0 1 0" />
     </joint>
     <link

Commit message: fix urdf contact frame & 4 legs kinematics

File: tinyquad_description/urdf/tinyquad_frame.urdf.xacro (robot description, xacro)
@@ -326,8 +326,4 @@
         effort="1.0787315"
         velocity="7.48" />
-      <!--mimic
-        joint="LFS_J"
-        multiplier="1"
-        offset="0" /-->
     </joint>
     <link
@@ -385,11 +381,7 @@
       <limit
         lower="0"
-        upper="1.1"
-        effort="1.0787315"
-        velocity="7.48" />
-      <!--mimic
-        joint="LFS_J"
-        multiplier="1"
-        offset="0" /-->
+        upper="1.4"
+        effort="1.0787315"
+        velocity="7.48" />
     </joint>
     <link
@@ -409,5 +401,5 @@
           izz="2.20437476815741E-05" />
       </inertial>
-      <!-- <visual>
+      <visual>
         <origin
           xyz="0 -0.0305 0"
@@ -431,5 +423,5 @@
             filename="package://tinyquad_description/meshes/RFL_L.STL" />
         </geometry>
-      </collision> -->
+      </collision>
     </link>
     <joint
@@ -446,12 +438,8 @@
         xyz="0 1 0" />
       <limit
-        lower="-1.5708"
-        upper="1.1"
-        effort="1.0787315"
-        velocity="7.48" />
-      <!--mimic
-        joint="LFS_J"
-        multiplier="1"
-        offset="0" /-->
+        lower="-1.8708"
+        upper="1.4"
+        effort="1.0787315"
+        velocity="7.48" />
     </joint>
     <link
@@ -473,38 +461,30 @@
       <visual>
         <origin
-          xyz="0 -0.0425 0"
-          rpy="0 0 0" />
-        <geometry>
-          <mesh
-            filename="package://tinyquad_description/meshes/RFC_L.STL" />
-        </geometry>
-        <material
-          name="">
-          <color
-            rgba="1 1 1 1" />
-        </material>
-      </visual>
-      <collision>
-        <origin
-          xyz="0 -0.0425 0"
-          rpy="0 0 0" />
-        <geometry>
-          <mesh
-            filename="package://tinyquad_description/meshes/RFC_L.STL" />
-        </geometry>
-      </collision>
-    </link>
-    <joint
-      name="RFC_J"
-      type="fixed">
-      <origin
-        xyz="1.9364E-05 0 -0.085"
-        rpy="0 0 0" />
-      <parent
-        link="RFL_L" />
-      <child
-        link="RFC_L" />
-      <axis
-        xyz="0 0 0" />
+          xyz="0 0.0425 0"
+          rpy="1.5708 0 0" />
+        <geometry>
+          <cylinder radius="0.001" length="0.01"/>
+        </geometry>
+        <material
+          name="">
+          <color
+            rgba="1 1 1 1" />
+        </material>
+      </visual>
+      <collision>
+        <origin
+          xyz="0 0.0425 0"
+          rpy="1.5708 0 0" />
+        <geometry>
+            <cylinder radius="0.001" length="0.1"/>
+        </geometry>
+      </collision>
+    </link>
+    <joint name="RFC_J" type="revolute">
+      <origin xyz="2.0629E-05 0 -0.085" rpy="0 0 0" />
+      <limit lower="-3.141592" upper="3.141592" effort="1.0787315" velocity="7.48" />
+      <parent link="RFL_L" />
+      <child link="RFC_L" />
+      <axis xyz="0 1 0" />
     </joint>
     <link
@@ -565,8 +545,4 @@
         effort="1.0787315"
         velocity="7.48" />
-      <!--mimic
-        joint="LFS_J"
-        multiplier="1"
-        offset="0" /-->
     </joint>
     <link
@@ -624,11 +600,7 @@
       <limit
         lower="0"
-        upper="1.1"
-        effort="1.0787315"
-        velocity="7.48" />
-      <!--mimic
-        joint="LFS_J"
-        multiplier="1"
-        offset="0" /-->
+        upper="1.4"
+        effort="1.0787315"
+        velocity="7.48" />
     </joint>
     <link
@@ -648,5 +620,5 @@
           izz="2.20436639521686E-05" />
       </inertial>
-      <!-- <visual>
+      <visual>
         <origin
           xyz="0 0.0305 0"
@@ -670,5 +642,5 @@
             filename="package://tinyquad_description/meshes/LBL_L.STL" />
         </geometry>
-      </collision> -->
+      </collision>
     </link>
     <joint
@@ -685,12 +657,8 @@
         xyz="0 1 0" />
       <limit
-        lower="-1.5708"
-        upper="1.1"
-        effort="1.0787315"
-        velocity="7.48" />
-      <!--mimic
-        joint="LFS_J"
-        multiplier="1"
-        offset="0" /-->
+        lower="-1.8708"
+        upper="1.4"
+        effort="1.0787315"
+        velocity="7.48" />
     </joint>
     <link
@@ -713,8 +681,7 @@
         <origin
           xyz="0 0.0425 0"
-          rpy="0 0 0" />
-        <geometry>
-          <mesh
-            filename="package://tinyquad_description/meshes/LBC_L.STL" />
+          rpy="1.5708 0 0" />
+        <geometry>
+          <cylinder radius="0.001" length="0.01"/>
         </geometry>
         <material
@@ -727,23 +694,16 @@
         <origin
           xyz="0 0.0425 0"
-          rpy="0 0 0" />
-        <geometry>
-          <mesh
-            filename="package://tinyquad_description/meshes/LBC_L.STL" />
-        </geometry>
-      </collision>
-    </link>
-    <joint
-      name="LBC_J"
-      type="fixed">
-      <origin
-        xyz="2.0629E-05 0 -0.085"
-        rpy="0 0 0" />
-      <parent
-        link="LBL_L" />
-      <child
-        link="LBC_L" />
-      <axis
-        xyz="0 0 0" />
+          rpy="1.5708 0 0" />
+        <geometry>
+            <cylinder radius="0.001" length="0.1"/>
+        </geometry>
+      </collision>
+    </link>
+    <joint name="LBC_J" type="revolute">
+      <origin xyz="2.0629E-05 0 -0.085" rpy="0 0 0" />
+      <limit lower="-3.141592" upper="3.141592" effort="1.0787315" velocity="7.48" />
+      <parent link="LBL_L" />
+      <child link="LBC_L" />
+      <axis xyz="0 1 0" />
     </joint>
     <link
@@ -804,8 +764,4 @@
         effort="1.0787315"
         velocity="7.48" />
-      <!--mimic
-        joint="LFS_J"
-        multiplier="1"
-        offset="0" /-->
     </joint>
     <link
@@ -863,11 +819,7 @@
       <limit
         lower="0"
-        upper="1.1"
-        effort="1.0787315"
-        velocity="7.48" />
-      <!--mimic
-        joint="LFS_J"
-        multiplier="1"
-        offset="0" /-->
+        upper="1.4"
+        effort="1.0787315"
+        velocity="7.48" />
     </joint>
     <link
@@ -887,5 +839,5 @@
           izz="2.20437476815741E-05" />
       </inertial>
-      <!-- <visual>
+      <visual>
         <origin
           xyz="0 -0.0305 0"
@@ -909,5 +861,5 @@
             filename="package://tinyquad_description/meshes/RBL_L.STL" />
         </geometry>
-      </collision> -->
+      </collision>
     </link>
     <joint
@@ -924,12 +876,8 @@
         xyz="0 1 0" />
       <limit
-        lower="-1.5708"
-        upper="1.1"
-        effort="1.0787315"
-        velocity="7.48" />
-      <!--mimic
-        joint="LFS_J"
-        multiplier="1"
-        offset="0" /-->
+        lower="-1.8708"
+        upper="1.4"
+        effort="1.0787315"
+        velocity="7.48" />
     </joint>
     <link
@@ -951,40 +899,31 @@
       <visual>
         <origin
-          xyz="0 -0.0425 0"
-          rpy="0 0 0" />
-        <geometry>
-          <mesh
-            filename="package://tinyquad_description/meshes/RBC_L.STL" />
-        </geometry>
-        <material
-          name="">
-          <color
-            rgba="1 1 1 1" />
-        </material>
-      </visual>
-      <collision>
-        <origin
-          xyz="0 -0.0425 0"
-          rpy="0 0 0" />
-        <geometry>
-          <mesh
-            filename="package://tinyquad_description/meshes/RBC_L.STL" />
-        </geometry>
-      </collision>
-    </link>
-    <joint
-      name="RBC_J"
-      type="fixed">
-      <origin
-        xyz="1.9364E-05 0 -0.085"
-        rpy="0 0 0" />
-      <parent
-        link="RBL_L" />
-      <child
-        link="RBC_L" />
-      <axis
-        xyz="0 0 0" />
+          xyz="0 0.0425 0"
+          rpy="1.5708 0 0" />
+        <geometry>
+          <cylinder radius="0.001" length="0.01"/>
+        </geometry>
+        <material
+          name="">
+          <color
+            rgba="1 1 1 1" />
+        </material>
+      </visual>
+      <collision>
+        <origin
+          xyz="0 0.0425 0"
+          rpy="1.5708 0 0" />
+        <geometry>
+            <cylinder radius="0.001" length="0.1"/>
+        </geometry>
+      </collision>
+    </link>
+    <joint name="RBC_J" type="revolute">
+      <origin xyz="2.0629E-05 0 -0.085" rpy="0 0 0" />
+      <limit lower="-3.141592" upper="3.141592" effort="1.0787315" velocity="7.48" />
+      <parent link="RBL_L" />
+      <child link="RBC_L" />
+      <axis xyz="0 1 0" />
     </joint>
   </xacro:macro>
-  <!-- <xacro:tinyquad_transmissions/> -->
 </robot>
