Commit message: refactor leg urdf xacro and add extra dof for trak ik and add tmux

File: tinyquad_description/urdf/tinyquad_frame.urdf.xacro (robot description, xacro)
@@ -1,4 +1,5 @@
 <?xml version="1.0"?>
 <robot xmlns:xacro="http://ros.org/wiki/xacro" >
+  <xacro:include filename="$(find tinyquad_description)/urdf/tinyquad_leg.xacro" />
   <xacro:macro name="tinyquad">
     <link name="base_footprint" >
@@ -50,880 +51,8 @@
       <child link="base_link" />
     </joint>
-    <link
-      name="LFS_L">
-      <inertial>
-        <origin
-          xyz="-0.046748 -0.00092972 6.6559E-07"
-          rpy="0 0 0" />
-        <mass
-          value="0.057684" />
-        <inertia
-          ixx="9.7817E-06"
-          ixy="5.1255E-07"
-          ixz="1.4506E-10"
-          iyy="1.4627E-05"
-          iyz="-7.3251E-10"
-          izz="1.8457E-05" />
-      </inertial>
-      <visual>
-        <origin
-          xyz="0 0 0"
-          rpy="0 0 0" />
-        <geometry>
-          <mesh
-            filename="package://tinyquad_description/meshes/LFS_L.STL" />
-        </geometry>
-        <material
-          name="">
-          <color
-            rgba="1 1 1 1" />
-        </material>
-      </visual>
-      <collision>
-        <origin
-          xyz="0 0 0"
-          rpy="0 0 0" />
-        <geometry>
-          <mesh
-            filename="package://tinyquad_description/meshes/LFS_L.STL" />
-        </geometry>
-      </collision>
-    </link>
-    <joint
-      name="LFS_J"
-      type="revolute">
-      <origin
-        xyz="0.15711 0.050443 0"
-        rpy="0 0 0" />
-      <parent
-        link="base_link" />
-      <child
-        link="LFS_L" />
-      <axis
-        xyz="1 0 0" />
-      <limit
-        lower="0"
-        upper="1.5708"
-        effort="1.0787315"
-        velocity="7.48" />
-    </joint>
-    <link
-      name="LFU_L">
-      <inertial>
-        <origin
-          xyz="0.00956780740114901 -0.00266058763780398 -0.0619406808382107"
-          rpy="0 0 0" />
-        <mass
-          value="0.0633248586799827" />
-        <inertia
-          ixx="4.22733905580439E-05"
-          ixy="-3.31314885518861E-08"
-          ixz="-4.35470998953999E-06"
-          iyy="3.42993494529219E-05"
-          iyz="4.30780434477683E-06"
-          izz="2.75949415936944E-05" />
-      </inertial>
-      <visual>
-        <origin
-          xyz="0 0.01375 0"
-          rpy="0 0 0" />
-        <geometry>
-          <mesh
-            filename="package://tinyquad_description/meshes/LFU_L.STL" />
-        </geometry>
-        <material
-          name="">
-          <color
-            rgba="1 1 1 1" />
-        </material>
-      </visual>
-      <collision>
-        <origin
-          xyz="0 0.01375 0"
-          rpy="0 0 0" />
-        <geometry>
-          <mesh
-            filename="package://tinyquad_description/meshes/LFU_L.STL" />
-        </geometry>
-      </collision>
-    </link>
-    <joint
-      name="LFU_J"
-      type="revolute">
-      <origin
-        xyz="-0.037107 0 0"
-        rpy="0 0 0" />
-      <parent
-        link="LFS_L" />
-      <child
-        link="LFU_L" />
-      <axis
-        xyz="0 1 0" />
-      <limit
-        lower="0"
-        upper="1.4"
-        effort="1.0787315"
-        velocity="7.48" />
-    </joint>
-    <link
-      name="LFL_L">
-      <inertial>
-        <origin
-          xyz="-0.0126991843001295 -0.0150723539446907 -0.0467923508835542"
-          rpy="0 0 0" />
-        <mass
-          value="0.0247326277403109" />
-        <inertia
-          ixx="4.21435291889056E-05"
-          ixy="4.52141590599905E-07"
-          ixz="2.40966499667341E-06"
-          iyy="2.82129703259535E-05"
-          iyz="1.66567501013991E-06"
-          izz="2.20436639521685E-05" />
-      </inertial>
-      <visual>
-        <origin
-          xyz="0 0.0305 0"
-          rpy="0 0 0" />
-        <geometry>
-          <mesh
-            filename="package://tinyquad_description/meshes/LFL_L.STL" />
-        </geometry>
-        <material
-          name="">
-          <color
-            rgba="1 1 1 1" />
-        </material>
-      </visual>
-      <collision>
-        <origin
-          xyz="0 0.0305 0"
-          rpy="0 0 0" />
-        <geometry>
-          <mesh
-            filename="package://tinyquad_description/meshes/LFL_L.STL" />
-        </geometry>
-      </collision>
-    </link>
-    <joint
-      name="LFL_J"
-      type="revolute">
-      <origin
-        xyz="0 0 -0.078388"
-        rpy="0 0 0" />
-      <parent
-        link="LFU_L" />
-      <child
-        link="LFL_L" />
-      <axis
-        xyz="0 1 0" />
-      <limit
-        lower="-1.8708"
-        upper="1.4"
-        effort="1.0787315"
-        velocity="7.48" />
-    </joint>
-    <link
-      name="LFC_L">
-      <inertial>
-        <origin
-          xyz="-0.0137408449020781 -0.0295642372944374 0.0344451912255238"
-          rpy="0 0 0" />
-        <mass
-          value="0.0228920746333247" />
-        <inertia
-          ixx="4.20984399971498E-05"
-          ixy="4.52141590599904E-07"
-          ixz="2.40966499667341E-06"
-          iyy="2.81277626908271E-05"
-          iyz="1.66567501013991E-06"
-          izz="2.19985747604127E-05" />
-      </inertial>
-      <visual>
-        <origin
-          xyz="0 0.0425 0"
-          rpy="1.5708 0 0" />
-        <geometry>
-          <cylinder radius="0.001" length="0.01"/>
-        </geometry>
-        <material
-          name="">
-          <color
-            rgba="1 1 1 1" />
-        </material>
-      </visual>
-      <collision>
-        <origin
-          xyz="0 0.0425 0"
-          rpy="1.5708 0 0" />
-        <geometry>
-            <cylinder radius="0.001" length="0.1"/>
-        </geometry>
-      </collision>
-    </link>
-    <joint name="LFC_J" type="revolute">
-      <origin xyz="2.0629E-05 0 -0.085" rpy="0 0 0" />
-      <limit lower="-3.141592" upper="3.141592" effort="1.0787315" velocity="7.48" />
-      <parent link="LFL_L" />
-      <child link="LFC_L" />
-      <axis xyz="0 1 0" />
-    </joint>
-    <link
-      name="RFS_L">
-      <inertial>
-        <origin
-          xyz="-0.0467477283228513 0.000929715895879799 -6.65623765903593E-07"
-          rpy="0 0 0" />
-        <mass
-          value="0.0576835055796688" />
-        <inertia
-          ixx="9.78169162854162E-06"
-          ixy="-5.12552767532585E-07"
-          ixz="-1.45029050660471E-10"
-          iyy="1.46267778399584E-05"
-          iyz="-7.32538517650851E-10"
-          izz="1.84573794225176E-05" />
-      </inertial>
-      <visual>
-        <origin
-          xyz="0 0 0"
-          rpy="0 0 0" />
-        <geometry>
-          <mesh
-            filename="package://tinyquad_description/meshes/RFS_L.STL" />
-        </geometry>
-        <material
-          name="">
-          <color
-            rgba="1 1 1 1" />
-        </material>
-      </visual>
-      <collision>
-        <origin
-          xyz="0 0 0"
-          rpy="0 0 0" />
-        <geometry>
-          <mesh
-            filename="package://tinyquad_description/meshes/RFS_L.STL" />
-        </geometry>
-      </collision>
-    </link>
-    <joint
-      name="RFS_J"
-      type="revolute">
-      <origin
-        xyz="0.15711 -0.050443 0"
-        rpy="0 0 0" />
-      <parent
-        link="base_link" />
-      <child
-        link="RFS_L" />
-      <axis
-        xyz="-1 0 0" />
-      <limit
-        lower="0"
-        upper="1.5708"
-        effort="1.0787315"
-        velocity="7.48" />
-    </joint>
-    <link
-      name="RFU_L">
-      <inertial>
-        <origin
-          xyz="0.00956728165308311 0.00266058760025918 -0.0619395881245908"
-          rpy="0 0 0" />
-        <mass
-          value="0.0633248589124594" />
-        <inertia
-          ixx="4.22736181545519E-05"
-          ixy="3.24961756510419E-08"
-          ixz="-4.35489106692463E-06"
-          iyy="3.42993499993469E-05"
-          iyz="-4.30648406795787E-06"
-          izz="2.75947147528143E-05" />
-      </inertial>
-      <visual>
-        <origin
-          xyz="0 -0.01375 0"
-          rpy="0 0 0" />
-        <geometry>
-          <mesh
-            filename="package://tinyquad_description/meshes/RFU_L.STL" />
-        </geometry>
-        <material
-          name="">
-          <color
-            rgba="0.898039215686275 0.917647058823529 0.929411764705882 1" />
-        </material>
-      </visual>
-      <collision>
-        <origin
-          xyz="0 -0.01375 0"
-          rpy="0 0 0" />
-        <geometry>
-          <mesh
-            filename="package://tinyquad_description/meshes/RFU_L.STL" />
-        </geometry>
-      </collision>
-    </link>
-    <joint
-      name="RFU_J"
-      type="revolute">
-      <origin
-        xyz="-0.037107 0 0"
-        rpy="0 0 0" />
-      <parent
-        link="RFS_L" />
-      <child
-        link="RFU_L" />
-      <axis
-        xyz="0 1 0" />
-      <limit
-        lower="0"
-        upper="1.4"
-        effort="1.0787315"
-        velocity="7.48" />
-    </joint>
-    <link
-      name="RFL_L">
-      <inertial>
-        <origin
-          xyz="-0.0127020493228516 0.0150724859124731 -0.0467927203950964"
-          rpy="0 0 0" />
-        <mass
-          value="0.0247329300871079" />
-        <inertia
-          ixx="4.21439137772161E-05"
-          ixy="-4.52171756192475E-07"
-          ixz="2.4097951023571E-06"
-          iyy="2.82133292880761E-05"
-          iyz="-1.66560968972201E-06"
-          izz="2.20437476815741E-05" />
-      </inertial>
-      <visual>
-        <origin
-          xyz="0 -0.0305 0"
-          rpy="0 0 0" />
-        <geometry>
-          <mesh
-            filename="package://tinyquad_description/meshes/RFL_L.STL" />
-        </geometry>
-        <material
-          name="">
-          <color
-            rgba="1 1 1 1" />
-        </material>
-      </visual>
-      <collision>
-        <origin
-          xyz="0 -0.0305 0"
-          rpy="0 0 0" />
-        <geometry>
-          <mesh
-            filename="package://tinyquad_description/meshes/RFL_L.STL" />
-        </geometry>
-      </collision>
-    </link>
-    <joint
-      name="RFL_J"
-      type="revolute">
-      <origin
-        xyz="0 0 -0.078391"
-        rpy="0 0 0" />
-      <parent
-        link="RFU_L" />
-      <child
-        link="RFL_L" />
-      <axis
-        xyz="0 1 0" />
-      <limit
-        lower="-1.8708"
-        upper="1.4"
-        effort="1.0787315"
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
File: tinyquad_description/urdf/tinyquad_leg.xacro (robot description, xacro)
@@ -5,5 +5,5 @@
         <inertial>
         <origin
-            xyz="-0.046748 ${y_mirror}*-0.00092972 6.6559E-07"
+            xyz="-0.046748 ${y_mirror*-0.00092972} 6.6559E-07"
             rpy="0 0 0" />
         <mass
@@ -11,8 +11,8 @@
         <inertia
             ixx="9.7817E-06"
-            ixy="${y_mirror}*${x_mirror}*5.1255E-07"
+            ixy="${y_mirror*x_mirror*5.1255E-07}"
             ixz="1.4506E-10"
             iyy="1.4627E-05"
-            iyz="${y_mirror}*-7.3251E-10"
+            iyz="${y_mirror*-7.3251E-10}"
             izz="1.8457E-05" />
         </inertial>
@@ -45,5 +45,5 @@
         type="revolute">
         <origin
-        xyz="0.15711-${x_offset} ${y_mirror}*0.050443 0"
+        xyz="${x_offset} ${y_mirror*0.050443} 0"
         rpy="0 0 0" />
         <parent
@@ -53,15 +53,24 @@
         <axis
         xyz="1 0 0" />
-        <limit
-        lower="0"
-        upper="1.5708"
-        effort="1.0787315"
-        velocity="7.48" />
-    </joint>
+        <xacro:if value="${y_mirror == 1}">
+            <limit
+            lower="-0.174533"
+            upper="1.5708"
+            effort="1.0787315"
+            velocity="7.48" />
+        </xacro:if>
+        <xacro:unless value="${y_mirror == 1}">
+            <limit
+            lower="-1.5708"
+            upper="0.174533"
+            effort="1.0787315"
+            velocity="7.48" />
+        </xacro:unless>
+        </joint>
     <link
         name="${pose_prefix}U_L">
         <inertial>
         <origin
-            xyz="0.00956780740114901 ${y_mirror}*-0.00266058763780398 -0.0619406808382107"
+            xyz="0.00956780740114901 ${y_mirror*-0.00266058763780398} -0.0619406808382107"
             rpy="0 0 0" />
         <mass
@@ -69,13 +78,13 @@
         <inertia
             ixx="4.22733905580439E-05"
-            ixy="${y_mirror}*${x_mirror}*-3.31314885518861E-08"
+            ixy="${y_mirror*x_mirror*-3.31314885518861E-08}"
             ixz="-4.35470998953999E-06"
             iyy="3.42993494529219E-05"
-            iyz="${y_mirror}*4.30780434477683E-06"
+            iyz="${y_mirror*4.30780434477683E-06}"
             izz="2.75949415936944E-05" />
         </inertial>
         <visual>
         <origin
-            xyz="0 ${y_mirror}*0.01375 0"
+            xyz="0 ${y_mirror*0.01375} 0"
             rpy="0 0 0" />
         <geometry>
@@ -91,5 +100,5 @@
         <collision>
         <origin
-            xyz="0 ${y_mirror}*0.01375 0"
+            xyz="0 ${y_mirror*0.01375} 0"
             rpy="0 0 0" />
         <geometry>
@@ -121,5 +130,5 @@
         <inertial>
         <origin
-            xyz="-0.0126991843001295 ${y_mirror}*-0.0150723539446907 -0.0467923508835542"
+            xyz="-0.0126991843001295 ${y_mirror*-0.0150723539446907} -0.0467923508835542"
             rpy="0 0 0" />
         <mass
@@ -127,13 +136,13 @@
         <inertia
             ixx="4.21435291889056E-05"
-            ixy="${y_mirror}*${x_mirror}*4.52141590599905E-07"
-            ixz="${x_mirror}*2.40966499667341E-06"
+            ixy="${y_mirror*x_mirror*4.52141590599905E-07}"
+            ixz="${x_mirror*2.40966499667341E-06}"
             iyy="2.82129703259535E-05"
-            iyz="${y_mirror}*1.66567501013991E-06"
+            iyz="${y_mirror*1.66567501013991E-06}"
             izz="2.20436639521685E-05" />
         </inertial>
         <visual>
         <origin
-            xyz="0 ${y_mirror}*0.0305 0"
+            xyz="0 ${y_mirror*0.0305} 0"
             rpy="0 0 0" />
         <geometry>
@@ -149,5 +158,5 @@
         <collision>
         <origin
-            xyz="0 ${y_mirror}*0.0305 0"
+            xyz="0 ${y_mirror*0.0305} 0"
             rpy="0 0 0" />
         <geometry>
@@ -179,5 +188,5 @@
         <inertial>
         <origin
-            xyz="-0.0137408449020781 ${y_mirror}*-0.0295642372944374 0.0344451912255238"
+            xyz="-0.0137408449020781 ${y_mirror*-0.0295642372944374} 0.0344451912255238"
             rpy="0 0 0" />
         <mass
@@ -185,8 +194,8 @@
         <inertia
             ixx="4.20984399971498E-05"
-            ixy="${y_mirror}*${x_mirror}*4.52141590599904E-07"
-            ixz="${x_mirror}*2.40966499667341E-06"
+            ixy="${y_mirror*x_mirror*4.52141590599904E-07}"
+            ixz="${x_mirror*2.40966499667341E-06}"
             iyy="2.81277626908271E-05"
-            iyz="${y_mirror}*1.66567501013991E-06"
+            iyz="${y_mirror*1.66567501013991E-06}"
             izz="2.19985747604127E-05" />
         </inertial>
@@ -223,4 +232,41 @@
         <axis xyz="0 1 0" />
     </joint>
+    <link
+    name="${pose_prefix}C2_L">
+      <inertial>
+        <origin
+          xyz="-0.0137408449020781 -0.0295642372944374 0.0344451912255238"
+          rpy="0 0 0" />
+        <mass
+          value="0.0228920746333247" />
+        <inertia
+          ixx="4.20984399971498E-05"
+          ixy="4.52141590599904E-07"
+          ixz="2.40966499667341E-06"
+          iyy="2.81277626908271E-05"
+          iyz="1.66567501013991E-06"
+          izz="2.19985747604127E-05" />
+      </inertial>
+      <visual>
+        <origin
+          xyz="0 0.0425 0"
+          rpy="0 1.5708 0" />
+        <geometry>
+          <cylinder radius="0.001" length="0.01"/>
+        </geometry>
+        <material
+          name="">
+          <color
+            rgba="1 1 1 1" />
+        </material>
+      </visual>
+    </link>
+    <joint name="${pose_prefix}C2_J" type="revolute">
+      <origin xyz="0 0 0" rpy="0 0 0" />
+      <limit lower="-3.141592" upper="3.141592" effort="1.0787315" velocity="7.48" />
+      <parent link="${pose_prefix}C_L" />
+      <child link="${pose_prefix}C2_L" />
+      <axis xyz="1 0 0" />
+    </joint>
   </xacro:macro>
 </robot>
