Commit message: init simple gait

File: tinyquad_description/urdf/tinyquad_leg.xacro (robot description, xacro)
@@ -200,5 +200,5 @@
             izz="2.19985747604127E-05" />
         </inertial>
-        <visual>
+        <!-- <visual>
         <origin
             xyz="0 0.0425 0"
@@ -212,5 +212,5 @@
             rgba="1 1 1 1" />
         </material>
-        </visual>
+        </visual> -->
         <collision>
         <origin
@@ -248,5 +248,5 @@
           izz="2.19985747604127E-05" />
       </inertial>
-      <visual>
+      <!-- <visual>
         <origin
           xyz="0 0.0425 0"
@@ -260,5 +260,5 @@
             rgba="1 1 1 1" />
         </material>
-      </visual>
+      </visual> -->
     </link>
     <joint name="${pose_prefix}C2_J" type="revolute">
